Commit message: Implemented new correct mesh files and measurements into the robot description files. Added configurable mounting points for the vertical sensor rail, and the angle of the lidar sensor. Camera to be implemented.

File: erwinia_os_description/urdf/amiga/amiga_macro.urdf.xacro (robot description, xacro)
@@ -4,23 +4,54 @@
         <!-- Build namespace prefix -->
         <xacro:property name="ns_prefix" value="${namespace}/${prefix}"/>
-        <!-- Wheel Mounting Positions -->
-        <xacro:property name="wheelbase" value="0.5316" />
-        <xacro:property name="track" value="0.65856" />
-        <!-- Wheel Properties -->
+        <!-- Wheel properties -->
+        <xacro:property name="wheel_z_offset" value="-0.393" /> <!-- Vertical offset of the wheel center from the base_link -->
+        <xacro:property name="wheelbase" value="0.77" /> <!-- Distance between front and rear wheel centers -->
+        <xacro:property name="track" value="0.98" /> <!-- Distance between left and right wheel centers (measured at the ground) -->
         <xacro:property name="wheel_radius" value="0.2159" />
+        <!-- Chasis properties -->
+        <xacro:property name="length" value="1.240" />
+        <xacro:property name="width" value="1.610" />
+        <xacro:property name="height_pos_z" value="1.181" /> <!-- Height from the base_link origin to the highest point of the robot -->
+        <xacro:property name="height_neg_z" value="${wheel_z_offset - wheel_radius}" /> <!-- Height from the base_link origin to the lowest point of the robot -->
+        <xacro:property name="height" value="${height_pos_z - height_neg_z}" /> <!-- Total height of the robot -->
+        <xacro:property name="bracket_top_height" value="0.353" />
+        <xacro:property name="imu_height" value="0.730" /> <!-- Height from the top of bracket to IMU mounting plate -->
+        <xacro:property name="lidar_height" value="0.657" /> <!-- Height from the top of bracket to lidar swivel bracket center -->
+        <xacro:property name="camera_height" value="0.4" /> <!-- Height from the top of bracket to camera swivel bracket center -->
+        <!-- Arm properties -->
+        <xacro:property name="arm_height" value="0.3212" /> <!-- Height from the top of bracket to IMU mounting plate -->
+        <!-- Collision properties -->
+        <xacro:property name="collision_buffer" value="0.05" /> <!-- Buffer added to a dimension of collision geometry dimensions for safety -->
+        <!-- Add in the main chassis/base_link -->
         <link name="${ns_prefix}base_link">
+            <inertial>
+                <origin xyz="-0.067 0.023 0.076" rpy="0 0 0" />
+                <mass value="456.0111243" />
+                <inertia ixx="154.11052182" ixy="6.17559451" ixz="18.36789382" iyy="127.1230648" iyz="-9.25081139" izz="162.24200762" />
+            </inertial>
             <visual>
-                <origin xyz="0 0 0" rpy="0 0 0" />
                 <geometry>
-                    <mesh filename="file://$(find erwinia_os_description)/meshes/frame_link.STL" />
+                    <mesh filename="file://$(find erwinia_os_description)/meshes/mid_level_asm.dae" />
                 </geometry>
-                <material name="">
-                    <color rgba="0.118 0.506 0.729 1" />
-                </material>
             </visual>
+            <!-- Lower chassis box -->
             <collision>
                 <origin xyz="0 0 0" rpy="0 0 0" />
                 <geometry>
-                    <mesh filename="file://$(find erwinia_os_description)/meshes/frame_collision.STL"  />
+                    <box size="${length + collision_buffer} ${width} ${arm_height*2 + collision_buffer}" />
+                </geometry>
+            </collision>
+            <!-- Upper body box -->
+            <collision>
+                <origin xyz="0 ${(1/6)*width} ${height_pos_z/2}" rpy="0 0 0" />
+                <geometry>
+                    <box size="${length + collision_buffer} ${(2/3)*width + collision_buffer} ${height_pos_z + collision_buffer}" />
+                </geometry>
+            </collision>
+            <!-- Display box -->
+            <collision>
+                <origin xyz="${-length/2} ${-width/4} ${height_pos_z/3}" rpy="0 0 0" />
+                <geometry>
+                    <box size="0.4 ${width/4 + collision_buffer} ${height_pos_z/4 + collision_buffer}" />
                 </geometry>
             </collision>
@@ -29,19 +60,73 @@
         <link name="${ns_prefix}base_footprint" />
         <joint name="${ns_prefix}base_footprint_joint" type="fixed">
+            <origin xyz="0 0 ${-wheel_z_offset + wheel_radius}" rpy="0 0 0" />
             <parent link="${ns_prefix}base_footprint" />
             <child link="${ns_prefix}base_link" />
         </joint>
-        <!-- Inertial link stores the robot's inertial information -->
-        <link name="${ns_prefix}inertial_link">
+        <!-- Positioning of the vertical rail holding the IMU -->
+        <link name="${ns_prefix}imu_mount">
             <inertial>
-                <mass value="381.19" />
-                <origin xyz="-0.054481 -0.015972 0.66252" />
-                <inertia ixx="5.717" ixy="-0.007109" ixz="0.0013622" iyy="12.857" iyz="1.2354E-05" izz="11.799" />
+                <origin xyz="0 0 -0.443" rpy="0 0 0" />
+                <mass value="3.431" />
+                <inertia ixx="0.26482927" ixy="0" ixz="0" iyy="0.26482927" iyz="0" izz="0.001" />
             </inertial>
+            <visual>
+                <geometry>
+                    <mesh filename="file://$(find erwinia_os_description)/meshes/vertical_rail.dae" />
+                </geometry>
+            </visual>
         </link>
-        <joint name="${ns_prefix}inertial_joint" type="fixed">
-            <origin xyz="0 0 0" rpy="0 0 0" />
+        <joint name="${ns_prefix}imu_mount_joint" type="fixed">
+            <origin xyz="0.032 -0.011 ${bracket_top_height + imu_height}" rpy="0 0 0" />
             <parent link="${ns_prefix}base_link" />
-            <child link="${ns_prefix}inertial_link" />
+            <child link="${ns_prefix}imu_mount" />
+        </joint>
+        <!-- Positioning of the swivel brackets -->
+        <!-- Lidar swivel bracket mount -->
+        <link name="${ns_prefix}swivel_bracket_lidar">
+            <visual>
+                <geometry>
+                    <mesh filename="file://$(find erwinia_os_description)/meshes/swivel_bracket.dae" />
+                </geometry>
+            </visual>
+        </link>
+        <joint name="${ns_prefix}swivel_bracket_lidar_joint" type="fixed">
+            <origin xyz="0.052 -0.011 ${bracket_top_height + lidar_height}" rpy="0 0 0" />
+            <parent link="${ns_prefix}base_link" />
+            <child link="${ns_prefix}swivel_bracket_lidar" />
+        </joint>
+        <!-- Lidar mount point — attach the lidar sensor here in a higher-level URDF -->
+        <link name="${ns_prefix}lidar_mount" />
+        <joint name="${ns_prefix}lidar_mount_joint" type="fixed">
+            <origin xyz="0.03 0 0" rpy="0 0 0" />
+            <parent link="${ns_prefix}swivel_bracket_lidar" />
+            <child link="${ns_prefix}lidar_mount" />
+        </joint>
+        <!-- Camera swivel bracket mount -->
+        <link name="${ns_prefix}swivel_bracket_camera">
+            <visual>
+                <geometry>
+                    <mesh filename="file://$(find erwinia_os_description)/meshes/swivel_bracket.dae" />
+                </geometry>
+            </visual>
+        </link>
+        <joint name="${ns_prefix}swivel_bracket_camera_joint" type="fixed">
+            <origin xyz="0.052 -0.011 ${bracket_top_height + camera_height}" rpy="0 0 0" />
+            <parent link="${ns_prefix}base_link" />
+            <child link="${ns_prefix}swivel_bracket_camera" />
+        </joint>
+        <!-- Camera mount point — attach the camera sensor here in a higher-level URDF -->
+        <link name="${ns_prefix}camera_mount" />
+        <joint name="${ns_prefix}camera_mount_joint" type="fixed">
+            <origin xyz="0.03 0 0" rpy="0 0 0" />
+            <parent link="${ns_prefix}swivel_bracket_camera" />
+            <child link="${ns_prefix}camera_mount" />
+        </joint>
+        <!-- arm mount -->
+        <link name="${ns_prefix}arm_mount" />
+        <joint name="${ns_prefix}arm_mount_joint" type="fixed">
+            <origin xyz="-0.02235400 -0.59689771 ${arm_height}" rpy="0 0 0" />
+            <parent link="${ns_prefix}base_link" />
+            <child link="${ns_prefix}arm_mount" />
         </joint>
         <!-- Amiga wheel macros -->
@@ -55,5 +140,5 @@
             <parent link="${ns_prefix}base_link"/>
             <child link="${ns_prefix}FL_wheel"/>
-            <origin xyz="${wheelbase/2} ${track/2} ${wheel_radius}" rpy="1.5708 0 3.1416" />
+            <origin xyz="${wheelbase/2} ${track/2} ${wheel_z_offset}" rpy="0 0 0" />
             <axis xyz="0 0 1" />
         </joint>
@@ -61,5 +146,5 @@
             <parent link="${ns_prefix}base_link"/>
             <child link="${ns_prefix}FR_wheel"/>
-            <origin xyz="${wheelbase/2} ${-track/2} ${wheel_radius}" rpy="1.5708 0 3.1416" />
+            <origin xyz="${wheelbase/2} ${-track/2} ${wheel_z_offset}" rpy="0 0 0" />
             <axis xyz="0 0 1" />
         </joint>
@@ -67,5 +152,5 @@
             <parent link="${ns_prefix}base_link"/>
             <child link="${ns_prefix}RL_wheel"/>
-            <origin xyz="${-wheelbase/2} ${track/2} ${wheel_radius}" rpy="1.5708 0 3.1416" />
+            <origin xyz="${-wheelbase/2} ${track/2} ${wheel_z_offset}" rpy="0 0 0" />
             <axis xyz="0 0 1" />
         </joint>
@@ -73,5 +158,5 @@
             <parent link="${ns_prefix}base_link"/>
             <child link="${ns_prefix}RR_wheel"/>
-            <origin xyz="${-wheelbase/2} ${-track/2} ${wheel_radius}" rpy="1.5708 0 3.1416" />
+            <origin xyz="${-wheelbase/2} ${-track/2} ${wheel_z_offset}" rpy="0 0 0" />
             <axis xyz="0 0 1" />
         </joint>

File: erwinia_os_description/urdf/amiga/amiga_wheel_macro.urdf.xacro (robot description, xacro)
@@ -4,21 +4,23 @@
         <link name="${wheel_prefix}_wheel">
             <inertial>
-                <origin xyz="4.3098E-07 5.5068E-07 -0.00020749" rpy="0 0 0" />
-                <mass value="15.628" />
-                <inertia ixx="0.153" ixy="1.1085E-06" ixz="2.7485E-07" iyy="0.153" iyz="2.341E-07" izz="0.28441" />
+                <origin xyz="-2.068e-7 -0.00020402 -1.642e-8" rpy="0 0 0" />
+                <mass value="15.62628337" />
+                <inertia
+                    ixx="0.15298774"
+                    ixy="-8.514e-7"
+                    ixz="1.530e-7"
+                    iyy="0.28438071"
+                    iyz="-7.993e-7"
+                    izz="0.15298827" />
             </inertial>
             <visual>
-                <origin xyz="0 0 0" rpy="0 0 0" />
                 <geometry>
-                    <mesh filename="file://$(find erwinia_os_description)/meshes/wheel.STL" />
+                    <mesh filename="file://$(find erwinia_os_description)/meshes/wheel.dae" />
                 </geometry>
-                <material name="">
-                    <color rgba="0 0 0 1" />
-                </material>
             </visual>
             <collision>
-                <origin xyz="0 0 0" rpy="0 0 0" />
+                <origin xyz="0 0 0" rpy="${pi/2} 0 0" />
                 <geometry>
-                    <mesh filename="file://$(find erwinia_os_description)/meshes/wheel_collision.STL" />
+                    <cylinder radius="0.2159" length="0.2" />
                 </geometry>
                 <!-- <surface>

File: erwinia_os_description/urdf/erwinia_os.urdf.xacro (robot description, xacro)
@@ -20,10 +20,11 @@
     <!-- TODO: Add in sensors with proper params-->
     <!-- SENSORS -->
+    <xacro:include filename="$(find erwinia_os_description)/urdf/sensors/amiga_lidar_macro.urdf.xacro"/>
+    <xacro:amiga_lidar
+        prefix="$(arg platform_ns)/$(arg platform_prefix)"
+        parent="$(arg platform_ns)/$(arg platform_prefix)lidar_mount"
+        angle_offset="${30.0 * (pi/180)}"/>
     <!-- <xacro:include filename="$(find erwinia_os_description)/urdf/sensors/amiga_camera_macro.urdf.xacro"/>
-    <xacro:include filename="$(find erwinia_os_description)/urdf/sensors/amiga_lidar_macro.urdf.xacro"/>
     <xacro:amiga_camera
-        prefix="$(arg platform_ns)/$(arg platform_prefix)"
-        parent="$(arg platform_ns)/$(arg platform_prefix)base_link"/>
-    <xacro:amiga_lidar
         prefix="$(arg platform_ns)/$(arg platform_prefix)"
         parent="$(arg platform_ns)/$(arg platform_prefix)base_link"/> -->
@@ -31,6 +32,6 @@
     <xacro:include filename="$(find erwinia_os_description)/urdf/xarm6/xarm6_macro.urdf.xacro"/>
     <xacro:xarm6 namespace="$(arg manipulator_ns)" prefix="$(arg manipulator_prefix)" model_num="1303"
-        parent_link="$(arg platform_ns)/$(arg platform_prefix)base_link">
-        <origin xyz="0.0 -0.8 1.0" rpy="0 0 ${-pi/2}"/>
+        parent_link="$(arg platform_ns)/$(arg platform_prefix)arm_mount">
+        <origin xyz="0 0 0" rpy="0 0 ${-pi/2}"/>
     </xacro:xarm6>
     <!-- ROS2_CONTROL -->

File: erwinia_os_description/urdf/sensors/amiga_lidar_macro.urdf.xacro (robot description, xacro)
@@ -1,25 +1,15 @@
 <?xml version="1.0" encoding="utf-8"?>
 <robot name="amiga_lidar" xmlns:xacro="http://www.ros.org/wiki/xacro">
-    <xacro:macro name="amiga_lidar" params="prefix:='' parent:='base_link'">
+    <xacro:macro name="amiga_lidar" params="prefix:='' parent:='lidar_mount' angle_offset:='0'">
         <!-- LIDAR -->
         <link name="${prefix}lidar_hinge">
-            <inertial>
-                <origin xyz="0.12957 -0.043305 -0.00024862" rpy="0 0 0" />
-                <mass value="5.5092" />
-                <inertia ixx="0.0061651" ixy="0.0013206" ixz="-1.4672E-06" iyy="0.0076386" iyz="1.274E-06" izz="0.0071961" />
-            </inertial>
             <visual>
-                <origin xyz="0 0 0" rpy="0 0 0" />
                 <geometry>
-                    <mesh filename="file://$(find erwinia_os_description)/meshes/lidar.STL" />
+                    <mesh filename="file://$(find erwinia_os_description)/meshes/lidar.dae" />
                 </geometry>
-                <material name="">
-                    <color rgba="0 1 0 1" />
-                </material>
             </visual>
         </link>
         <joint name="${prefix}lidar_hinge_joint" type="fixed">
-            <origin xyz="1.1572 0.18502 1.449" rpy="1.5708 -0.4363 0" />
-            <!-- change pitch to adjust camera angle. + is down.  -0.4363 makes it parallel to ground -->
+            <origin xyz="0 0 0" rpy="0 ${angle_offset} 0" />
             <parent link="${parent}" />
             <child link="${prefix}lidar_hinge" />
@@ -27,9 +17,7 @@
         <link name="${prefix}lidar" />
         <joint name="${prefix}lidar_joint" type="fixed">
-            <origin xyz="0.14354 -0.042185 0" rpy="-1.5708 0 -0.43633" />
-            <!-- 0.82903 applied in ypr order -->
+            <origin xyz="0.14791768 0 0.02247100" rpy="0 0 0" />
             <parent link="${prefix}lidar_hinge" />
             <child link="${prefix}lidar" />
-            <axis xyz="0 0 0" />
         </joint>
         <!-- GAZEBO LIDAR SENSOR PLUGIN -->

Commit message: Fixed issues with dae models not showing up in gazebo. Converted models to low-res objs for compute (gutted electronics and screws). Fixed wheel rotation axis. Works in gazebo now.

File: erwinia_os_description/urdf/amiga/amiga_macro.urdf.xacro (robot description, xacro)
@@ -32,5 +32,5 @@
             <visual>
                 <geometry>
-                    <mesh filename="file://$(find erwinia_os_description)/meshes/mid_level_asm.dae" />
+                    <mesh filename="file://$(find erwinia_os_description)/meshes/mid_level_asm/mid_level_asm.obj" />
                 </geometry>
             </visual>
@@ -73,5 +73,5 @@
             <visual>
                 <geometry>
-                    <mesh filename="file://$(find erwinia_os_description)/meshes/vertical_rail.dae" />
+                    <mesh filename="file://$(find erwinia_os_description)/meshes/vertical_rail/vertical_rail.obj" />
                 </geometry>
             </visual>
@@ -87,5 +87,5 @@
             <visual>
                 <geometry>
-                    <mesh filename="file://$(find erwinia_os_description)/meshes/swivel_bracket.dae" />
+                    <mesh filename="file://$(find erwinia_os_description)/meshes/swivel_bracket/swivel_bracket.obj" />
                 </geometry>
             </visual>
@@ -107,5 +107,5 @@
             <visual>
                 <geometry>
-                    <mesh filename="file://$(find erwinia_os_description)/meshes/swivel_bracket.dae" />
+                    <mesh filename="file://$(find erwinia_os_description)/meshes/swivel_bracket/swivel_bracket.obj" />
                 </geometry>
             </visual>
@@ -141,5 +141,5 @@
             <child link="${ns_prefix}FL_wheel"/>
             <origin xyz="${wheelbase/2} ${track/2} ${wheel_z_offset}" rpy="0 0 0" />
-            <axis xyz="0 0 1" />
+            <axis xyz="0 1 0" />
         </joint>
         <joint name="${ns_prefix}FR_wheel_joint" type="continuous">
@@ -147,5 +147,5 @@
             <child link="${ns_prefix}FR_wheel"/>
             <origin xyz="${wheelbase/2} ${-track/2} ${wheel_z_offset}" rpy="0 0 0" />
-            <axis xyz="0 0 1" />
+            <axis xyz="0 1 0" />
         </joint>
         <joint name="${ns_prefix}RL_wheel_joint" type="continuous">
@@ -153,5 +153,5 @@
             <child link="${ns_prefix}RL_wheel"/>
             <origin xyz="${-wheelbase/2} ${track/2} ${wheel_z_offset}" rpy="0 0 0" />
-            <axis xyz="0 0 1" />
+            <axis xyz="0 1 0" />
         </joint>
         <joint name="${ns_prefix}RR_wheel_joint" type="continuous">
@@ -159,5 +159,5 @@
             <child link="${ns_prefix}RR_wheel"/>
             <origin xyz="${-wheelbase/2} ${-track/2} ${wheel_z_offset}" rpy="0 0 0" />
-            <axis xyz="0 0 1" />
+            <axis xyz="0 1 0" />
         </joint>
     </xacro:macro>

File: erwinia_os_description/urdf/amiga/amiga_wheel_macro.urdf.xacro (robot description, xacro)
@@ -16,5 +16,5 @@
             <visual>
                 <geometry>
-                    <mesh filename="file://$(find erwinia_os_description)/meshes/wheel.dae" />
+                    <mesh filename="file://$(find erwinia_os_description)/meshes/wheel/wheel.obj" />
                 </geometry>
             </visual>

File: erwinia_os_description/urdf/sensors/amiga_lidar_macro.urdf.xacro (robot description, xacro)
@@ -6,5 +6,5 @@
             <visual>
                 <geometry>
-                    <mesh filename="file://$(find erwinia_os_description)/meshes/lidar.dae" />
+                    <mesh filename="file://$(find erwinia_os_description)/meshes/lidar/lidar.obj" />
                 </geometry>
             </visual>
