Commit message: Updated the wheel names in the control pkg and removed the platform controller from the real-world launch (only launches with use_gazebo:=true).

File: erwinia_os_description/urdf/amiga/amiga_ros2_control.xacro (robot description, xacro)
@@ -25,5 +25,5 @@
     </xacro:macro>
     <xacro:macro name="amiga_system_joints" params="prefix">
-        <joint name="${prefix}FL_wheel_joint">
+        <joint name="${prefix}front_left_wheel_joint">
             <command_interface name="velocity">
                 <param name="min">-2.54</param>
@@ -33,5 +33,5 @@
             <state_interface name="velocity"/>
         </joint>
-        <joint name="${prefix}FR_wheel_joint">
+        <joint name="${prefix}front_right_wheel_joint">
             <command_interface name="velocity">
                 <param name="min">-2.54</param>
@@ -41,5 +41,5 @@
             <state_interface name="velocity"/>
         </joint>
-        <joint name="${prefix}RL_wheel_joint">
+        <joint name="${prefix}rear_left_wheel_joint">
             <command_interface name="velocity">
                 <param name="min">-2.54</param>
@@ -49,5 +49,5 @@
             <state_interface name="velocity"/>
         </joint>
-        <joint name="${prefix}RR_wheel_joint">
+        <joint name="${prefix}rear_right_wheel_joint">
             <command_interface name="velocity">
                 <param name="min">-2.54</param>
