Commit message: Updated the srdf to remove adjacent collisions and updated the wheel names in the urdf to match.

File: erwinia_os_description/srdf/erwinia_os.srdf.xacro (robot description, xacro)
@@ -36,7 +36,6 @@
         <joint name="${arm_prefix}joint6" value="0"/>
     </group_state>
-    <!-- <xacro:include filename="$(find multi_camera_rig_description)/srdf/multi_cam_rig.srdf.xacro"/> -->
-    <!-- <xacro:multi_camera_rig/> -->
-    <!-- TODO: Add in collision matrix -->
+    <xacro:include filename="$(find multi_camera_rig_description)/srdf/multi_cam_rig.srdf.xacro"/>
+    <xacro:multi_camera_rig/>
     <disable_collisions link1="${arm_prefix}link1" link2="${arm_prefix}link2" reason="Adjacent"/>
     <disable_collisions link1="${arm_prefix}link1" link2="${arm_prefix}link3" reason="Never"/>
@@ -48,16 +47,12 @@
     <disable_collisions link1="${arm_prefix}link5" link2="${arm_prefix}link6" reason="Adjacent"/>
     <disable_collisions link1="${arm_prefix}base_link" link2="${base_prefix}base_link" reason="Never"/>
-    <!-- <disable_collisions link1="${arm_prefix}base_link" link2="${base_prefix}top_chassis_link" reason="Default"/>
     <disable_collisions link1="${arm_prefix}base_link" link2="${base_prefix}front_left_wheel" reason="Never"/>
     <disable_collisions link1="${arm_prefix}base_link" link2="${base_prefix}front_right_wheel" reason="Never"/>
     <disable_collisions link1="${arm_prefix}base_link" link2="${base_prefix}rear_left_wheel" reason="Never"/>
     <disable_collisions link1="${arm_prefix}base_link" link2="${base_prefix}rear_right_wheel" reason="Never"/>
-    <disable_collisions link1="${arm_prefix}base_link" link2="${base_prefix}x_rail_riser_link" reason="Adjacent"/>
-    <disable_collisions link1="${arm_prefix}link1" link2="${base_prefix}x_rail_riser_link" reason="Never"/>
     <disable_collisions link1="${base_prefix}base_link" link2="${base_prefix}front_left_wheel" reason="Adjacent"/>
     <disable_collisions link1="${base_prefix}base_link" link2="${base_prefix}front_right_wheel" reason="Adjacent"/>
     <disable_collisions link1="${base_prefix}base_link" link2="${base_prefix}rear_left_wheel" reason="Adjacent"/>
     <disable_collisions link1="${base_prefix}base_link" link2="${base_prefix}rear_right_wheel" reason="Adjacent"/>
-    <disable_collisions link1="${base_prefix}base_link" link2="${base_prefix}x_rail_riser_link" reason="Adjacent"/>
-    <disable_collisions link1="${arm_prefix}link6" link2="multi_camera_rig_link" reason="Adjacent"/> -->
+    <disable_collisions link1="${arm_prefix}link6" link2="multi_camera_rig_link" reason="Adjacent"/>
 </robot>

File: erwinia_os_description/urdf/amiga/amiga_macro.urdf.xacro (robot description, xacro)
@@ -132,30 +132,30 @@
         <!-- Amiga wheel macros -->
         <xacro:include filename="$(find erwinia_os_description)/urdf/amiga/amiga_wheel_macro.urdf.xacro" />
-        <xacro:amiga_wheel wheel_prefix="${ns_prefix}FL" use_gazebo="${use_gazebo}" />
-        <xacro:amiga_wheel wheel_prefix="${ns_prefix}FR" use_gazebo="${use_gazebo}" />
-        <xacro:amiga_wheel wheel_prefix="${ns_prefix}RL" use_gazebo="${use_gazebo}" />
-        <xacro:amiga_wheel wheel_prefix="${ns_prefix}RR" use_gazebo="${use_gazebo}" />
+        <xacro:amiga_wheel wheel_prefix="${ns_prefix}front_left" use_gazebo="${use_gazebo}" />
+        <xacro:amiga_wheel wheel_prefix="${ns_prefix}front_right" use_gazebo="${use_gazebo}" />
+        <xacro:amiga_wheel wheel_prefix="${ns_prefix}rear_left" use_gazebo="${use_gazebo}" />
+        <xacro:amiga_wheel wheel_prefix="${ns_prefix}rear_right" use_gazebo="${use_gazebo}" />
         <!-- Define wheel joints to use prefixed base_link -->
-        <joint name="${ns_prefix}FL_wheel_joint" type="continuous">
+        <joint name="${ns_prefix}front_left_wheel_joint" type="continuous">
             <parent link="${ns_prefix}base_link"/>
-            <child link="${ns_prefix}FL_wheel"/>
+            <child link="${ns_prefix}front_left_wheel"/>
             <origin xyz="${wheelbase/2} ${track/2} ${wheel_z_offset}" rpy="0 0 0" />
             <axis xyz="0 1 0" />
         </joint>
-        <joint name="${ns_prefix}FR_wheel_joint" type="continuous">
+        <joint name="${ns_prefix}front_right_wheel_joint" type="continuous">
             <parent link="${ns_prefix}base_link"/>
-            <child link="${ns_prefix}FR_wheel"/>
+            <child link="${ns_prefix}front_right_wheel"/>
             <origin xyz="${wheelbase/2} ${-track/2} ${wheel_z_offset}" rpy="0 0 0" />
             <axis xyz="0 1 0" />
         </joint>
-        <joint name="${ns_prefix}RL_wheel_joint" type="continuous">
+        <joint name="${ns_prefix}rear_left_wheel_joint" type="continuous">
             <parent link="${ns_prefix}base_link"/>
-            <child link="${ns_prefix}RL_wheel"/>
+            <child link="${ns_prefix}rear_left_wheel"/>
             <origin xyz="${-wheelbase/2} ${track/2} ${wheel_z_offset}" rpy="0 0 0" />
             <axis xyz="0 1 0" />
         </joint>
-        <joint name="${ns_prefix}RR_wheel_joint" type="continuous">
+        <joint name="${ns_prefix}rear_right_wheel_joint" type="continuous">
             <parent link="${ns_prefix}base_link"/>
-            <child link="${ns_prefix}RR_wheel"/>
+            <child link="${ns_prefix}rear_right_wheel"/>
             <origin xyz="${-wheelbase/2} ${-track/2} ${wheel_z_offset}" rpy="0 0 0" />
             <axis xyz="0 1 0" />
