Commit message: Added xarm to the description package (temporary positioning).

File: erwinia_os_description/urdf/erwinia_os.urdf.xacro (robot description, xacro)
@@ -9,4 +9,6 @@
     <xacro:arg name="platform_ns" default="amiga"/>
     <xacro:arg name="platform_prefix" default=""/>
+    <xacro:arg name="manipulator_ip" default="192.168.1.205"/>
+    <xacro:arg name="report_type" default="normal"/>
     <!-- TODO: Fine tune Amiga model -->
     <!-- AMIGA PLATFORM -->
@@ -26,6 +28,12 @@
         prefix="$(arg platform_ns)/$(arg platform_prefix)"
         parent="$(arg platform_ns)/$(arg platform_prefix)base_link"/> -->
-    <!-- TODO: Add in robotic manipulator -->
+    <!-- xArm6 Robotic Manipulator -->
+    <xacro:include filename="$(find husky_xarm6_mcr_description)/urdf/xarm6/xarm6_macro.urdf.xacro"/>
+    <xacro:xarm6 namespace="$(arg manipulator_ns)" prefix="$(arg manipulator_prefix)" model_num="1303"
+        parent_link="$(arg platform_ns)/$(arg platform_prefix)base_link">
+        <origin xyz="0.0 -0.8 1.0" rpy="0 0 ${-pi/2}"/>
+    </xacro:xarm6>
     <!-- ROS2_CONTROL -->
+    <!-- Controller config for the Amiga platform -->
     <xacro:include filename="$(find erwinia_os_description)/urdf/amiga/amiga_ros2_control.xacro"/>
     <xacro:amiga_ros2_control
@@ -34,4 +42,13 @@
         use_gazebo="$(arg use_gazebo)"
         use_fake_hardware="$(arg use_fake_hardware)"/>
+    <!-- Controller config for the xArm6 manipulator -->
+    <xacro:include filename="$(find husky_xarm6_mcr_description)/urdf/xarm6/xarm6_ros2_control.xacro"/>
+    <xacro:xarm6_ros2_control
+        namespace="$(arg manipulator_ns)"
+        prefix="$(arg manipulator_prefix)"
+        use_gazebo="$(arg use_gazebo)"
+        use_fake_hardware="$(arg use_fake_hardware)"
+        robot_ip="$(arg manipulator_ip)"
+        report_type="$(arg report_type)"/>
     <!-- Gazebo plugin for controller manager (only needed once for whole robot) -->
     <xacro:if value="$(arg use_gazebo)">

Commit message: Updated the dependencies and the urdf to include the multi camera rig.

File: erwinia_os_description/urdf/erwinia_os.urdf.xacro (robot description, xacro)
@@ -35,4 +35,12 @@
         <origin xyz="0 0 0" rpy="0 0 ${-pi/2}"/>
     </xacro:xarm6>
+    <!-- MULTI CAMERA RIG -->
+    <xacro:include filename="$(find multi_camera_rig_description)/urdf/multi_camera_rig_macro.urdf.xacro"/>
+    <xacro:multi_camera_rig use_gazebo="$(arg use_gazebo)"/>
+    <joint name="tool_mount" type="fixed">
+        <parent link="$(arg manipulator_ns)/$(arg manipulator_prefix)link_eef"/>
+        <child link="multi_camera_rig_mount"/>
+        <origin xyz="0.0 0.0 0.0" rpy="${pi/2} 0 0"/>
+    </joint>
     <!-- ROS2_CONTROL -->
     <!-- Controller config for the Amiga platform -->

Commit message: Yi navigation bulk commit.

File: erwinia_os_description/urdf/erwinia_os.urdf.xacro (robot description, xacro)
@@ -22,12 +22,17 @@
     <xacro:include filename="$(find erwinia_os_description)/urdf/sensors/amiga_lidar_macro.urdf.xacro"/>
     <xacro:amiga_lidar
-        prefix="$(arg platform_ns)/$(arg platform_prefix)"
+        prefix=""
         parent="$(arg platform_ns)/$(arg platform_prefix)lidar_mount"
-        angle_offset="${30.0 * (pi/180)}"/>
+        angle_offset="${24.0 * (pi/180)}"/>
     <xacro:include filename="$(find erwinia_os_description)/urdf/sensors/amiga_gnss_macro.urdf.xacro"/>
     <xacro:amiga_gnss
-        prefix="$(arg platform_ns)/$(arg platform_prefix)"
+        prefix=""
         parent="$(arg platform_ns)/$(arg platform_prefix)imu_mount"
         z_offset="0.019"/>
+    <xacro:include filename="$(find erwinia_os_description)/urdf/sensors/amiga_imu_macro.urdf.xacro"/>
+    <xacro:amiga_imu
+        prefix="vectornav/"
+        parent="$(arg platform_ns)/$(arg platform_prefix)imu_mount"
+        z_offset="0.005"/>
     <!-- <xacro:include filename="$(find erwinia_os_description)/urdf/sensors/amiga_camera_macro.urdf.xacro"/>
     <xacro:amiga_camera

File: erwinia_os_description/urdf/sensors/amiga_gnss_macro.urdf.xacro (robot description, xacro)
@@ -12,5 +12,5 @@
         <link name="${prefix}gnss">
             <visual>
-                <origin xyz="0 0 0" rpy="${pi/2} 0 ${pi/2}" />
+                <origin xyz="0 0 0" rpy="${pi/2} 0 ${-pi/2}" />
                 <geometry>
                     <mesh filename="file://$(find erwinia_os_description)/meshes/gnss/gnss.obj" />

File: erwinia_os_description/urdf/sensors/amiga_lidar_macro.urdf.xacro (robot description, xacro)
@@ -15,12 +15,12 @@
             <child link="${prefix}lidar_hinge" />
         </joint>
-        <link name="${prefix}lidar" />
+        <link name="${prefix}velodyne" />
         <joint name="${prefix}lidar_joint" type="fixed">
             <origin xyz="0.14791768 0 0.02247100" rpy="0 0 0" />
             <parent link="${prefix}lidar_hinge" />
-            <child link="${prefix}lidar" />
+            <child link="${prefix}velodyne" />
         </joint>
         <!-- GAZEBO LIDAR SENSOR PLUGIN -->
-        <gazebo reference="${prefix}lidar">
+        <gazebo reference="${prefix}velodyne">
             <sensor name="gpu_lidar" type="gpu_lidar">
                 <!-- block_laser_sensor might work for 3d? -->
@@ -56,5 +56,5 @@
                 <always_on>1</always_on>
                 <visualize>true</visualize>
-                <gz_frame_id>${prefix}lidar</gz_frame_id>
+                <gz_frame_id>${prefix}velodyne</gz_frame_id>
             </sensor>
         </gazebo>
