Commit message: Added xarm collapsed and zero positions.

File: common/erwinia_os_description/srdf/erwinia_os.srdf.xacro (robot description, xacro)
@@ -28,10 +28,18 @@
         <joint name="${arm_prefix}joint6" value="1.5708"/>
     </group_state>
-    <group_state name="hold-up" group="xarm6_manipulator">
+    <group_state name="collapsed" group="xarm6_manipulator">
+        <joint name="${arm_prefix}joint1" value="1.5708"/>
+        <joint name="${arm_prefix}joint2" value="-1.5708"/>
+        <joint name="${arm_prefix}joint3" value="0"/>
+        <joint name="${arm_prefix}joint4" value="0"/>
+        <joint name="${arm_prefix}joint5" value="0"/>
+        <joint name="${arm_prefix}joint6" value="1.5708"/>
+    </group_state>
+    <group_state name="zero" group="xarm6_manipulator">
         <joint name="${arm_prefix}joint1" value="0"/>
         <joint name="${arm_prefix}joint2" value="0"/>
         <joint name="${arm_prefix}joint3" value="0"/>
         <joint name="${arm_prefix}joint4" value="0"/>
-        <joint name="${arm_prefix}joint5" value="-1.5708"/>
+        <joint name="${arm_prefix}joint5" value="0"/>
         <joint name="${arm_prefix}joint6" value="0"/>
     </group_state>

Commit message: calib pose added.

File: common/erwinia_os_description/srdf/erwinia_os.srdf.xacro (robot description, xacro)
@@ -22,4 +22,12 @@
     <group_state name="home" group="xarm6_manipulator">
         <joint name="${arm_prefix}joint1" value="0.0"/>
+        <joint name="${arm_prefix}joint2" value="-0.7854"/>
+        <joint name="${arm_prefix}joint3" value="-0.7854"/>
+        <joint name="${arm_prefix}joint4" value="0.0"/>
+        <joint name="${arm_prefix}joint5" value="0.0"/>
+        <joint name="${arm_prefix}joint6" value="1.5708"/>
+    </group_state>
+    <group_state name="calib" group="xarm6_manipulator">
+        <joint name="${arm_prefix}joint1" value="-1.5708"/>
         <joint name="${arm_prefix}joint2" value="-0.7854"/>
         <joint name="${arm_prefix}joint3" value="-0.7854"/>

Commit message: Updated the demo and action server planners to use a set of initial joint configurations designed to prevent arm collisions.

File: common/erwinia_os_description/srdf/erwinia_os.srdf.xacro (robot description, xacro)
@@ -22,6 +22,8 @@
     <group_state name="home" group="xarm6_manipulator">
         <joint name="${arm_prefix}joint1" value="0.0"/>
-        <joint name="${arm_prefix}joint2" value="-0.7854"/>
-        <joint name="${arm_prefix}joint3" value="-0.7854"/>
+        <!-- <joint name="${arm_prefix}joint2" value="-0.7854"/> -->
+        <joint name="${arm_prefix}joint2" value="-0.34906585"/>
+        <!-- <joint name="${arm_prefix}joint3" value="-0.7854"/> -->
+        <joint name="${arm_prefix}joint3" value="-1.22173048"/>
         <joint name="${arm_prefix}joint4" value="0.0"/>
         <joint name="${arm_prefix}joint5" value="0.0"/>
